File: ECE4900_Senior_Thesis.kicad_sch (KiCad schematic)
At the start: 87 parts, among them J1 1757242, J2 1757242, J3 Conn_02x10_Odd_Even, J4 Conn_01x04, Q1 CSD18540Q5B, Q2 CSD18540Q5B, Q3 Q_PMOS_GSD, Q4 CSD18540Q5B, SW1 SW_Push, U1 UCC27301ADR, U2 TPS7A1601QDGNRQ1, U3 STM32G474CBT6TR, U4 LMR51610XDBVR, U5 INA240A2DR, U6 INA240A2DR, U7 LM74700QDBVRQ1

Commit message: Add files via upload
{RESC6432X90N.kicad_mod
IND_1273AS-H-220M=P3.kicad_mod
D8_TEX.kicad_mod
DBV0006A-IPC_A.kicad_mod
DGN8_1P92X1P6_TEX.kicad_mod
CSD18540Q5B.kicad_mod
UCC27301ADR.kicad_mod} - go into FloatingPV.pretty
Parts:
- C1: footprint (none) -> Capacitor_SMD:CP_Elec_8x6.9
- C10, C13, C4, C5, C9: footprint (none) -> Capacitor_SMD:C_1210_3225Metric
- C11, C14, C15, C16, C17, C19, C20, C21, C22, C23, C24, C25, C26, C27, C28, C29, C30, C6, C7: footprint (none) -> Capacitor_SMD:C_0603_1608Metric
- C12: footprint (none) -> Capacitor_SMD:C_1206_3216Metric
- C18, C8: footprint (none) -> Capacitor_SMD:C_0805_2012Metric
- C2, C3: footprint (none) -> Capacitor_SMD:CP_Elec_10x12.5
- F1, F2: footprint (none) -> Fuse:Fuse_Littelfuse-NANO2-451_453
- FB1: footprint (none) -> Inductor_SMD:L_0603_1608Metric
- J1, J2: footprint (none) -> Connector_Phoenix_MSTB:PhoenixContact_MSTBA_2,5_2-G-5,08_1x02_P5.08mm_Horizontal
- J3: footprint (none) -> Connector_IDC:IDC-Header_2x10_P2.54mm_Vertical
- J4: footprint (none) -> Connector_PinHeader_2.54mm:PinHeader_1x04_P2.54mm_Vertical
- L2: footprint (none) -> FloatingPV:IND_1273AS-H-220M=P3
- LED1: footprint (none) -> LED_SMD:LED_0603_1608Metric
- Q3: footprint (none) -> Package_SON:Diodes_PowerDI3333-8
- R1, R2: footprint (none) -> Resistor_SMD:R_0805_2012Metric
- R10, R11, R12, R13, R14, R15, R16, R17, R18, R19, R3, R4, R5, R6, R7, R8, R9, TH1: footprint (none) -> Resistor_SMD:R_0603_1608Metric
- RSH2: footprint (none) -> FloatingPV:RESC6432X90N
- SW1: footprint (none) -> Button_Switch_THT:SW_PUSH_6mm_H4.3mm
- TP1, TP10, TP11, TP2, TP3, TP4, TP5, TP6, TP7, TP8, TP9: footprint (none) -> TestPoint:TestPoint_Keystone_5000-5004_Miniature
- TVS1: footprint Diode_SMD:D_0805_2012Metric -> Diode_SMD:D_SMB
- U2: footprint DGN8_1P92X1P6_TEX -> FloatingPV:DGN8_1P92X1P6_TEX
- U4: footprint DBV0006A-IPC_A -> FloatingPV:DBV0006A-IPC_A
- ZD1: footprint (none) -> Diode_SMD:D_SOD-123
