File: ECE4900_Senior_Thesis.kicad_sch (KiCad schematic)
At the start: 75 parts, among them J1 1757242, J2 1757242, J3 Conn_02x10_Odd_Even, J4 Conn_01x04, Q1 CSD18540Q5B, Q2 CSD18540Q5B, Q3 Q_PMOS_GSD, Q4 CSD18540Q5B, SW1 SW_Push, U1 UCC27301ADR, U2 TPS7A1601QDGNRQ1, U3 STM32G474CBT6TR, U4 LMR51610XDBVR, U5 INA240A2DR, U6 INA240A2DR, U7 LM74700QDBVRQ1

Commit message: Finalized schematic and began assigning footprints
Parts:
- added LED1: LED, symbol Device:LED
- added R19: 1kΩ, symbol Device:R
- added TP10, TP11, TP2, TP3, TP4, TP5, TP6, TP7, TP8, TP9: TestPoint, symbol Connector:TestPoint
- F2: value 0451007.MRL -> 0451010.MRL
- Q1, Q2, Q4: footprint DNK0008A -> FloatingPV:CSD18540Q5B
- R12: value 10k -> 10kΩ
- RSH2: value 10mΩ -> 5mΩ
- TVS1: value SMBJ33A -> SMBJ28A
- U1: footprint SOIC8_D_TEX -> FloatingPV:UCC27301ADR
Connections:
- net +12V_AUX: now also TP7.1
- net +3V3: now also C13.1, TP8.1; no longer C13.2
- net BAT_OUT: now also TP6.1
- net BUCK_OUT: now also TP5.1
- net GND: now also C13.2, Q2.3 (Source), LED1.1 (K), TP9.1; no longer C13.1
- net PV_BUS: now also TP4.1
- net PV_IN: now also TP2.1
- net PV_PROTECTED: now also TP3.1
- net PWM_HI: now also TP10.1
- net PWM_LI: now also TP11.1
- net at R4.1: now also Q2.2 (Gate), R2.1; no longer Q2.3 (Source)
- net at U3.42 (PB5): now also R19.2
- new net: LED1.2 (A), R19.1
- no-connect marks 9 -> 29
Other:
- note added: "DEBUGGING"
- note added: "INPUT PROTECTION"
- note added: "OUTPUT PROTECTION"
- moved on the sheet: C13, R4

Commit message: Preliminary Layout Finished
Further pre-fab inspection is neccessary
Parts:
- removed L1: 22uH, symbol Device:L
- added L1: 22 uH, FloatingPV:CSCF2014-220MC, symbol CSCF2014-220MC:CSCF2014-220MC
- C1: footprint (none) -> Capacitor_SMD:CP_Elec_8x6.9; KiLib_Generator (none) -> capacitor/SMD/elec_round_polarized
- C10, C13, C4, C5, C9: footprint (none) -> Capacitor_SMD:C_1210_3225Metric; KiLib_Generator (none) -> SMD_2terminal_chip_molded
- C11, C14, C15, C16, C17, C19, C20, C21, C22, C23, C24, C25, C26, C27, C28, C29, C30, C6, C7: footprint (none) -> Capacitor_SMD:C_0603_1608Metric; KiLib_Generator (none) -> SMD_2terminal_chip_molded
- C12: footprint (none) -> Capacitor_SMD:C_1206_3216Metric; KiLib_Generator (none) -> SMD_2terminal_chip_molded
- C18, C8: footprint (none) -> Capacitor_SMD:C_0805_2012Metric; KiLib_Generator (none) -> SMD_2terminal_chip_molded
- C2, C3: footprint (none) -> Capacitor_SMD:CP_Elec_10x12.5; KiLib_Generator (none) -> capacitor/SMD/elec_round_polarized
- F1, F2: footprint (none) -> Fuse:Fuse_Littelfuse-NANO2-451_453
- FB1: footprint (none) -> Inductor_SMD:L_0603_1608Metric; KiLib_Generator (none) -> SMD_2terminal_chip_molded
- J1, J2: footprint (none) -> Connector_Phoenix_MSTB:PhoenixContact_MSTBA_2,5_2-G-5,08_1x02_P5.08mm_Horizontal; KiLib_Generator (none) -> connector/PhoenixContact
- J3: footprint (none) -> Connector_IDC:IDC-Header_2x10_P2.54mm_Vertical; KiLib_Generator (none) -> connector/pin_header_socket
- J4: footprint (none) -> Connector_PinHeader_2.54mm:PinHeader_1x04_P2.54mm_Vertical; KiLib_Generator (none) -> connector/pin_header_socket
- L2: footprint (none) -> FloatingPV:IND_1273AS-H-220M=P3
- LED1: footprint (none) -> LED_SMD:LED_0603_1608Metric; KiLib_Generator (none) -> SMD_2terminal_chip_molded
- Q3: footprint (none) -> Package_SON:Diodes_PowerDI3333-8
- R1, R2: footprint (none) -> Resistor_SMD:R_0805_2012Metric; KiLib_Generator (none) -> SMD_2terminal_chip_molded
- R10, R11, R12, R13, R14, R15, R16, R17, R18, R19, R3, R4, R5, R6, R7, R8, R9, TH1: footprint (none) -> Resistor_SMD:R_0603_1608Metric; KiLib_Generator (none) -> SMD_2terminal_chip_molded
- RSH1: footprint (none) -> FloatingPV:KRL3264E-C-R010-F-T1
- RSH2: footprint (none) -> FloatingPV:RESC6432X90N
- SW1: footprint (none) -> Button_Switch_THT:SW_PUSH_6mm_H4.3mm
- TP1, TP10, TP11, TP2, TP3, TP4, TP5, TP6, TP7, TP8, TP9: footprint (none) -> TestPoint:TestPoint_Keystone_5000-5004_Miniature
- TVS1: footprint Diode_SMD:D_0805_2012Metric -> Diode_SMD:D_SMB
- U2: footprint DGN8_1P92X1P6_TEX -> FloatingPV:DGN8_1P92X1P6_TEX
- U3, U5, U6, U7: KiLib_Generator (none) -> package/gullwing
- U4: footprint DBV0006A-IPC_A -> FloatingPV:DBV0006A-IPC_A
- ZD1: footprint (none) -> Diode_SMD:D_SOD-123
Connections:
- net BUCK_OUT: now also L1.2
- net SW: now also C6.2, U1.4 (HS), L1.1
Other:
- moved on the sheet: C1, F2, Q1, Q2, R2, R3, R4, TP5
